Commit message: new version

File: description/robot.urdf.xacro (robot description, xacro)
@@ -2,4 +2,7 @@
 <robot xmlns:xacro="http://www.ros.org/wiki/xacro"  name="robot">
     <xacro:include filename="robot_core.xacro" />
-   <xacro:include filename="gazebo_control.xacro" />
+    <!-- <xacro:include filename="gazebo_control.xacro" /> -->
+    <xacro:include filename="ros2_control.xacro" />
+    <xacro:include filename="lidar.xacro" />
+    <xacro:include filename="camera.xacro" />
 </robot>

File: description/robot_core.xacro (robot description, xacro)
@@ -13,4 +13,7 @@
     <material name="black">
         <color rgba="0 0 0 1"/>
+    </material>
+     <material name="red">
+        <color rgba="1 0 0 1"/>
     </material>
     <link name="base_link">
@@ -59,5 +62,5 @@
         <collision>
             <geometry>
-                <cylinder length="0.04" radius="0.05" />/>
+                <sphere radius="0.05" />/>
             </geometry>
         </collision>
@@ -85,5 +88,5 @@
         <collision>
             <geometry>
-                <cylinder length="0.04" radius="0.05" />/>
+                <sphere radius="0.05" />/>
             </geometry>
         </collision>
